Commit message: built a basic robot in rover package

File: Rover/description/rover_core.xacro (robot description, xacro)
@@ -1,4 +1,5 @@
 <?xml version="1.0"?>
 <robot xmlns:xacro="http://www.ros.org/wiki/xacro" >
+    <xacro:include filename="inertial_macros.xacro"/>
     <!-- BASE LINK -->
     <link name="base_link">
@@ -16,5 +17,4 @@
                 <box size="0.3 0.3 0.15"/>
             </geometry>
-            <material name="white"/>
         </visual>
         <collision>
@@ -25,5 +25,5 @@
         </collision>
         <xacro:inertial_box mass="0.5" x="0.3" y="0.3" z="0.15">
-            <origin xyz="0.15 0 0.075" rpy="0 0 0"/>
+            <origin xyz="0.15 0.0 0.075"/>
         </xacro:inertial_box>
     </link>
@@ -41,4 +41,55 @@
             </geometry>
         </visual>
+        <collision>
+            <geometry>
+                <cylinder radius="0.05" length="0.04"/>
+            </geometry>
+        </collision>
+        <xacro:inertial_cylinder mass="0.1" length="0.04" radius="0.05">
+            <origin xyz="0.0 0.0 0.0"/>
+        </xacro:inertial_cylinder>
+    </link>
+    <!-- RIGHT WHEEL LINK -->
+    <joint name="right_wheel_joint" type="continuous">
+        <parent link="base_link"/>
+        <child link="right_wheel_link"/>
+        <origin xyz="0 -0.175 0" rpy="${pi/2} 0 0" />
+        <axis xyz="0 0 -1"/>
+    </joint>
+    <link name="right_wheel_link">
+        <visual>
+            <geometry>
+                <cylinder radius="0.05" length="0.04"/>
+            </geometry>
+        </visual>
+        <collision>
+            <geometry>
+                <cylinder radius="0.05" length="0.04"/>
+            </geometry>
+        </collision>
+        <xacro:inertial_cylinder mass="0.1" length="0.04" radius="0.05">
+            <origin xyz="0.0 0.0 0.0"/>
+        </xacro:inertial_cylinder>
+    </link>
+    <!-- CASTER WHEEL LINK -->
+    <joint name="caster_wheel_joint" type = "fixed">
+        <parent link="chassis"/>
+        <child link="caster_wheel"/>
+        <origin xyz="0.24 0.0 0.0"/>
+    </joint>
+    <link name="caster_wheel">
+        <visual>
+            <geometry>
+                <sphere radius="0.05"/>
+            </geometry>
+        </visual>
+        <collision>
+            <geometry>
+                <sphere radius="0.05"/>
+            </geometry>
+        </collision>
+        <xacro:inertial_sphere mass="0.1" radius="0.05">
+            <origin xyz="0.0 0.0 0.0"/>
+        </xacro:inertial_sphere>
     </link>
 </robot>
