Commit message: using package:// insted of file://

File: Manipulator/description/manipulator_core.xacro (robot description, xacro)
@@ -26,5 +26,5 @@
       <geometry>
         <mesh
-          filename="file://$(find arm2)/meshes/base_link.STL" />
+          filename="package://arm2/meshes/base_link.STL" />
       </geometry>
       <material
@@ -40,5 +40,5 @@
       <geometry>
         <mesh
-          filename="file://$(find arm2)/meshes/base_link.STL" />
+          filename="package://arm2/meshes/base_link.STL" />
       </geometry>
     </collision>
@@ -66,5 +66,5 @@
       <geometry>
         <mesh
-          filename="file://$(find arm2)/meshes/link1.STL" />
+          filename="package://arm2/meshes/link1.STL" />
       </geometry>
       <material
@@ -80,5 +80,5 @@
       <geometry>
         <mesh
-          filename="file://$(find arm2)/meshes/link1.STL" />
+          filename="package://arm2/meshes/link1.STL" />
       </geometry>
     </collision>
@@ -119,5 +119,5 @@
       <geometry>
         <mesh
-          filename="file://$(find arm2)/meshes/link2.STL" />
+          filename="package://arm2/meshes/link2.STL" />
       </geometry>
       <material
@@ -133,5 +133,5 @@
       <geometry>
         <mesh
-          filename="file://$(find arm2)/meshes/link2.STL" />
+          filename="package://arm2/meshes/link2.STL" />
       </geometry>
     </collision>
@@ -172,5 +172,5 @@
       <geometry>
         <mesh
-          filename="file://$(find arm2)/meshes/link3.STL" />
+          filename="package://arm2/meshes/link3.STL" />
       </geometry>
       <material
@@ -186,5 +186,5 @@
       <geometry>
         <mesh
-          filename="file://$(find arm2)/meshes/link3.STL" />
+          filename="package://arm2/meshes/link3.STL" />
       </geometry>
     </collision>
@@ -225,5 +225,5 @@
       <geometry>
         <mesh
-          filename="file://$(find arm2)/meshes/link4.STL" />
+          filename="package://arm2/meshes/link4.STL" />
       </geometry>
       <material
@@ -239,5 +239,5 @@
       <geometry>
         <mesh
-          filename="file://$(find arm2)/meshes/link4.STL" />
+          filename="package://arm2/meshes/link4.STL" />
       </geometry>
     </collision>
@@ -278,5 +278,5 @@
       <geometry>
         <mesh
-          filename="file://$(find arm2)/meshes/link5.STL" />
+          filename="package://arm2/meshes/link5.STL" />
       </geometry>
       <material
@@ -292,5 +292,5 @@
       <geometry>
         <mesh
-          filename="file://$(find arm2)/meshes/link5.STL" />
+          filename="package://arm2/meshes/link5.STL" />
       </geometry>
     </collision>
@@ -331,5 +331,5 @@
       <geometry>
         <mesh
-          filename="file://$(find arm2)/meshes/link6.STL" />
+          filename="package://arm2/meshes/link6.STL" />
       </geometry>
       <material
@@ -345,5 +345,5 @@
       <geometry>
         <mesh
-          filename="file://$(find arm2)/meshes/link6.STL" />
+          filename="package://arm2/meshes/link6.STL" />
       </geometry>
     </collision>
@@ -384,5 +384,5 @@
       <geometry>
         <mesh
-          filename="file://$(find arm2)/meshes/link7.STL" />
+          filename="package://arm2/meshes/link7.STL" />
       </geometry>
       <material
@@ -398,5 +398,5 @@
       <geometry>
         <mesh
-          filename="file://$(find arm2)/meshes/link7.STL" />
+          filename="package://arm2/meshes/link7.STL" />
       </geometry>
     </collision>

File: assem1_description/urdf/assem1.urdf.xacro (robot description, xacro)
@@ -13,5 +13,5 @@
     <origin xyz="0 0 0" rpy="0 0 0"/>
     <geometry>
-      <mesh filename="file://$(find assem1_description)/meshes/base_link.STL" scale="0.001 0.001 0.001"/>
+      <mesh filename="package://assem1_description/meshes/base_link.STL" scale="0.001 0.001 0.001"/>
     </geometry>
     <material name="silver"/>
@@ -20,5 +20,5 @@
     <origin xyz="0 0 0" rpy="0 0 0"/>
     <geometry>
-      <mesh filename="file://$(find assem1_description)/meshes/base_link.STL" scale="0.001 0.001 0.001"/>
+      <mesh filename="package://assem1_description/meshes/base_link.STL" scale="0.001 0.001 0.001"/>
     </geometry>
   </collision>
@@ -33,5 +33,5 @@
     <origin xyz="0.003063 -0.003089 -0.190919" rpy="0 0 0"/>
     <geometry>
-      <mesh filename="file://$(find assem1_description)/meshes/Part2_1.STL" scale="0.001 0.001 0.001"/>
+      <mesh filename="package://assem1_description/meshes/Part2_1.STL" scale="0.001 0.001 0.001"/>
     </geometry>
     <material name="silver"/>
@@ -40,5 +40,5 @@
     <origin xyz="0.003063 -0.003089 -0.190919" rpy="0 0 0"/>
     <geometry>
-      <mesh filename="file://$(find assem1_description)/meshes/Part2_1.STL" scale="0.001 0.001 0.001"/>
+      <mesh filename="package://assem1_description/meshes/Part2_1.STL" scale="0.001 0.001 0.001"/>
     </geometry>
   </collision>
@@ -53,5 +53,5 @@
     <origin xyz="0.038331 0.142706 -0.330919" rpy="0 0 0"/>
     <geometry>
-      <mesh filename="file://$(find assem1_description)/meshes/Part3_1.STL" scale="0.001 0.001 0.001"/>
+      <mesh filename="package://assem1_description/meshes/Part3_1.STL" scale="0.001 0.001 0.001"/>
     </geometry>
     <material name="silver"/>
@@ -60,5 +60,5 @@
     <origin xyz="0.038331 0.142706 -0.330919" rpy="0 0 0"/>
     <geometry>
-      <mesh filename="file://$(find assem1_description)/meshes/Part3_1.STL" scale="0.001 0.001 0.001"/>
+      <mesh filename="package://assem1_description/meshes/Part3_1.STL" scale="0.001 0.001 0.001"/>
     </geometry>
   </collision>
@@ -73,5 +73,5 @@
     <origin xyz="-0.030387 -0.141374 -0.523471" rpy="0 0 0"/>
     <geometry>
-      <mesh filename="file://$(find assem1_description)/meshes/Part4_1.STL" scale="0.001 0.001 0.001"/>
+      <mesh filename="package://assem1_description/meshes/Part4_1.STL" scale="0.001 0.001 0.001"/>
     </geometry>
     <material name="silver"/>
@@ -80,5 +80,5 @@
     <origin xyz="-0.030387 -0.141374 -0.523471" rpy="0 0 0"/>
     <geometry>
-      <mesh filename="file://$(find assem1_description)/meshes/Part4_1.STL" scale="0.001 0.001 0.001"/>
+      <mesh filename="package://assem1_description/meshes/Part4_1.STL" scale="0.001 0.001 0.001"/>
     </geometry>
   </collision>
@@ -93,5 +93,5 @@
     <origin xyz="-0.004873 0.081066 -0.584516" rpy="0 0 0"/>
     <geometry>
-      <mesh filename="file://$(find assem1_description)/meshes/Part5_1.STL" scale="0.001 0.001 0.001"/>
+      <mesh filename="package://assem1_description/meshes/Part5_1.STL" scale="0.001 0.001 0.001"/>
     </geometry>
     <material name="silver"/>
@@ -100,5 +100,5 @@
     <origin xyz="-0.004873 0.081066 -0.584516" rpy="0 0 0"/>
     <geometry>
-      <mesh filename="file://$(find assem1_description)/meshes/Part5_1.STL" scale="0.001 0.001 0.001"/>
+      <mesh filename="package://assem1_description/meshes/Part5_1.STL" scale="0.001 0.001 0.001"/>
     </geometry>
   </collision>
@@ -113,5 +113,5 @@
     <origin xyz="0.003681 0.20663 -0.638292" rpy="0 0 0"/>
     <geometry>
-      <mesh filename="file://$(find assem1_description)/meshes/Part7_1.STL" scale="0.001 0.001 0.001"/>
+      <mesh filename="package://assem1_description/meshes/Part7_1.STL" scale="0.001 0.001 0.001"/>
     </geometry>
     <material name="silver"/>
@@ -120,5 +120,5 @@
     <origin xyz="0.003681 0.20663 -0.638292" rpy="0 0 0"/>
     <geometry>
-      <mesh filename="file://$(find assem1_description)/meshes/Part7_1.STL" scale="0.001 0.001 0.001"/>
+      <mesh filename="package://assem1_description/meshes/Part7_1.STL" scale="0.001 0.001 0.001"/>
     </geometry>
   </collision>
@@ -133,5 +133,5 @@
     <origin xyz="-0.023282 0.148493 -0.723368" rpy="0 0 0"/>
     <geometry>
-      <mesh filename="file://$(find assem1_description)/meshes/Part8_1.STL" scale="0.001 0.001 0.001"/>
+      <mesh filename="package://assem1_description/meshes/Part8_1.STL" scale="0.001 0.001 0.001"/>
     </geometry>
     <material name="silver"/>
@@ -140,5 +140,5 @@
     <origin xyz="-0.023282 0.148493 -0.723368" rpy="0 0 0"/>
     <geometry>
-      <mesh filename="file://$(find assem1_description)/meshes/Part8_1.STL" scale="0.001 0.001 0.001"/>
+      <mesh filename="package://assem1_description/meshes/Part8_1.STL" scale="0.001 0.001 0.001"/>
     </geometry>
   </collision>
@@ -153,5 +153,5 @@
     <origin xyz="-0.059773 0.120751 -0.715132" rpy="0 0 0"/>
     <geometry>
-      <mesh filename="file://$(find assem1_description)/meshes/Part9_1.STL" scale="0.001 0.001 0.001"/>
+      <mesh filename="package://assem1_description/meshes/Part9_1.STL" scale="0.001 0.001 0.001"/>
     </geometry>
     <material name="green"/>
@@ -160,5 +160,5 @@
     <origin xyz="-0.059773 0.120751 -0.715132" rpy="0 0 0"/>
     <geometry>
-      <mesh filename="file://$(find assem1_description)/meshes/Part9_1.STL" scale="0.001 0.001 0.001"/>
+      <mesh filename="package://assem1_description/meshes/Part9_1.STL" scale="0.001 0.001 0.001"/>
     </geometry>
   </collision>
@@ -173,5 +173,5 @@
     <origin xyz="-0.019773 0.1530751 -0.765132" rpy="0 0 0"/>
     <geometry>
-      <mesh filename="file://$(find assem1_description)/meshes/Part9_2.STL" scale="0.001 0.001 0.001"/>
+      <mesh filename="package://assem1_description/meshes/Part9_2.STL" scale="0.001 0.001 0.001"/>
     </geometry>
     <material name="red"/>
@@ -180,5 +180,5 @@
     <origin xyz="-0.606893 -0.042637 -0.23854" rpy="0 0 0"/>
     <geometry>
-      <mesh filename="file://$(find assem1_description)/meshes/Part9_2.STL" scale="0.001 0.001 0.001"/>
+      <mesh filename="package://assem1_description/meshes/Part9_2.STL" scale="0.001 0.001 0.001"/>
     </geometry>
   </collision>
@@ -193,5 +193,5 @@
     <origin xyz="0.003063 -0.003089 -0.085919" rpy="0 0 0"/>
     <geometry>
-      <mesh filename="file://$(find assem1_description)/meshes/Part1_1.STL" scale="0.001 0.001 0.001"/>
+      <mesh filename="package://assem1_description/meshes/Part1_1.STL" scale="0.001 0.001 0.001"/>
     </geometry>
     <material name="silver"/>
@@ -200,5 +200,5 @@
     <origin xyz="0.003063 -0.003089 -0.085919" rpy="0 0 0"/>
     <geometry>
-      <mesh filename="file://$(find assem1_description)/meshes/Part1_1.STL" scale="0.001 0.001 0.001"/>
+      <mesh filename="package://assem1_description/meshes/Part1_1.STL" scale="0.001 0.001 0.001"/>
     </geometry>
   </collision>
@@ -213,5 +213,5 @@
     <origin xyz="-0.236937 0.316911 -0.005919" rpy="0 0 0"/>
     <geometry>
-      <mesh filename="file://$(find assem1_description)/meshes/wheel_v1_1.STL" scale="0.001 0.001 0.001"/>
+      <mesh filename="package://assem1_description/meshes/wheel_v1_1.STL" scale="0.001 0.001 0.001"/>
     </geometry>
     <material name="silver"/>
@@ -220,5 +220,5 @@
     <origin xyz="-0.236937 0.316911 -0.005919" rpy="0 0 0"/>
     <geometry>
-      <mesh filename="file://$(find assem1_description)/meshes/wheel_v1_1.STL" scale="0.001 0.001 0.001"/>
+      <mesh filename="package://assem1_description/meshes/wheel_v1_1.STL" scale="0.001 0.001 0.001"/>
     </geometry>
   </collision>
@@ -233,5 +233,5 @@
     <origin xyz="-0.236937 -0.323089 -0.005919" rpy="0 0 0"/>
     <geometry>
-      <mesh filename="file://$(find assem1_description)/meshes/wheel_v1__1__1.STL" scale="0.001 0.001 0.001"/>
+      <mesh filename="package://assem1_description/meshes/wheel_v1__1__1.STL" scale="0.001 0.001 0.001"/>
     </geometry>
     <material name="silver"/>
@@ -240,5 +240,5 @@
     <origin xyz="-0.236937 -0.323089 -0.005919" rpy="0 0 0"/>
     <geometry>
-      <mesh filename="file://$(find assem1_description)/meshes/wheel_v1__1__1.STL" scale="0.001 0.001 0.001"/>
+      <mesh filename="package://assem1_description/meshes/wheel_v1__1__1.STL" scale="0.001 0.001 0.001"/>
     </geometry>
   </collision>
@@ -253,5 +253,5 @@
     <origin xyz="0.243063 -0.323089 -0.005919" rpy="0 0 0"/>
     <geometry>
-      <mesh filename="file://$(find assem1_description)/meshes/wheel_v1__2__1.STL" scale="0.001 0.001 0.001"/>
+      <mesh filename="package://assem1_description/meshes/wheel_v1__2__1.STL" scale="0.001 0.001 0.001"/>
     </geometry>
     <material name="silver"/>
@@ -260,5 +260,5 @@
     <origin xyz="0.243063 -0.323089 -0.005919" rpy="0 0 0"/>
     <geometry>
-      <mesh filename="file://$(find assem1_description)/meshes/wheel_v1__2__1.STL" scale="0.001 0.001 0.001"/>
+      <mesh filename="package://assem1_description/meshes/wheel_v1__2__1.STL" scale="0.001 0.001 0.001"/>
     </geometry>
   </collision>
@@ -273,5 +273,5 @@
     <origin xyz="0.243063 0.316911 -0.005919" rpy="0 0 0"/>
     <geometry>
-      <mesh filename="file://$(find assem1_description)/meshes/wheel_v1__3__1.STL" scale="0.001 0.001 0.001"/>
+      <mesh filename="package://assem1_description/meshes/wheel_v1__3__1.STL" scale="0.001 0.001 0.001"/>
     </geometry>
     <material name="silver"/>
@@ -280,5 +280,5 @@
     <origin xyz="0.243063 0.316911 -0.005919" rpy="0 0 0"/>
     <geometry>
-      <mesh filename="file://$(find assem1_description)/meshes/wheel_v1__3__1.STL" scale="0.001 0.001 0.001"/>
+      <mesh filename="package://assem1_description/meshes/wheel_v1__3__1.STL" scale="0.001 0.001 0.001"/>
     </geometry>
   </collision>
@@ -293,5 +293,5 @@
     <origin xyz="0.003063 0.316911 -0.045919" rpy="0 0 0"/>
     <geometry>
-      <mesh filename="file://$(find assem1_description)/meshes/camera_1.STL" scale="0.001 0.001 0.001"/>
+      <mesh filename="package://assem1_description/meshes/camera_1.STL" scale="0.001 0.001 0.001"/>
     </geometry>
     <material name="silver"/>
@@ -300,5 +300,5 @@
     <origin xyz="0.003063 0.316911 -0.045919" rpy="0 0 0"/>
     <geometry>
-      <mesh filename="file://$(find assem1_description)/meshes/camera_1.STL" scale="0.001 0.001 0.001"/>
+      <mesh filename="package://assem1_description/meshes/camera_1.STL" scale="0.001 0.001 0.001"/>
     </geometry>
   </collision>
@@ -313,5 +313,5 @@
     <origin xyz="0.006126 0.313823 -0.091838" rpy="0 0 0"/>
     <geometry>
-      <mesh filename="file://$(find assem1_description)/meshes/lidar_1.STL" scale="0.001 0.001 0.001"/>
+      <mesh filename="package://assem1_description/meshes/lidar_1.STL" scale="0.001 0.001 0.001"/>
     </geometry>
     <material name="silver"/>
@@ -320,5 +320,5 @@
     <origin xyz="0.006126 0.313823 -0.091838" rpy="0 0 0"/>
     <geometry>
-      <mesh filename="file://$(find assem1_description)/meshes/lidar_1.STL" scale="0.001 0.001 0.001"/>
+      <mesh filename="package://assem1_description/meshes/lidar_1.STL" scale="0.001 0.001 0.001"/>
     </geometry>
   </collision>
