Commit message: revolute_8 origin changed

File: assem1_description/urdf/assem1.urdf.xacro (robot description, xacro)
@@ -155,5 +155,5 @@
       <mesh filename="file://$(find assem1_description)/meshes/Part9_1.STL" scale="0.001 0.001 0.001"/>
     </geometry>
-    <material name="silver"/>
+    <material name="green"/>
   </visual>
   <collision>
@@ -171,9 +171,9 @@
   </inertial>
   <visual>
-    <origin xyz="-0.606893 -0.042637 -0.23854" rpy="0 0 0"/>
+    <origin xyz="-0.019773 0.1530751 -0.765132" rpy="0 0 0"/>
     <geometry>
       <mesh filename="file://$(find assem1_description)/meshes/Part9_2.STL" scale="0.001 0.001 0.001"/>
     </geometry>
-    <material name="silver"/>
+    <material name="red"/>
   </visual>
   <collision>
@@ -371,5 +371,5 @@
 </joint>
 <joint name="Revolute 8" type="revolute">
-  <origin xyz="0.583611 0.19113 -0.484828" rpy="0 0 0"/>
+  <origin xyz="-0.01 -0.01 0.04" rpy="0 0 0"/>
   <parent link="Part8_1"/>
   <child link="Part9_2"/>

Commit message: colour change

File: assem1_description/urdf/assem1.urdf.xacro (robot description, xacro)
@@ -155,5 +155,5 @@
       <mesh filename="package://assem1_description/meshes/Part9_1.STL" scale="0.001 0.001 0.001"/>
     </geometry>
-    <material name="green"/>
+    <material name="silver"/>
   </visual>
   <collision>
@@ -175,5 +175,5 @@
       <mesh filename="package://assem1_description/meshes/Part9_2.STL" scale="0.001 0.001 0.001"/>
     </geometry>
-    <material name="red"/>
+    <material name="silver"/>
   </visual>
   <collision>

Commit message: fixed wheel direction

File: assem1_description/urdf/assem1.urdf.xacro (robot description, xacro)
@@ -397,5 +397,5 @@
   <parent link="base_link"/>
   <child link="wheel_v1__2__1"/>
-  <axis xyz="-1.0 0.0 0.0"/>
+  <axis xyz="1.0 0.0 0.0"/>
 </joint>
 <joint name="Revolute 13" type="continuous">
@@ -403,5 +403,5 @@
   <parent link="base_link"/>
   <child link="wheel_v1__3__1"/>
-  <axis xyz="-1.0 0.0 0.0"/>
+  <axis xyz="1.0 0.0 0.0"/>
 </joint>
 <joint name="Rigid 16" type="fixed">

Commit message: added lidar

File: assem1_description/urdf/assem1.urdf.xacro (robot description, xacro)
@@ -3,4 +3,5 @@
 <xacro:include filename="$(find assem1_description)/urdf/materials.xacro" />
 <xacro:include filename="$(find assem1_description)/urdf/assem1.gazebo" />
+<xacro:include filename="$(find assem1_description)/urdf/lidar.xacro"/>
 <link name="base_link">
   <inertial>
@@ -300,24 +301,4 @@
     <geometry>
       <mesh filename="file://$(find assem1_description)/meshes/camera_1.STL" scale="0.001 0.001 0.001"/>
-    </geometry>
-  </collision>
-</link>
-<link name="lidar_1">
-  <inertial>
-    <origin xyz="0.003062764224799069 0.036911727731188615 0.014080953287975456" rpy="0 0 0"/>
-    <mass value="0.3945840372908781"/>
-    <inertia ixx="9.2e-05" iyy="9.2e-05" izz="7.9e-05" ixy="-0.0" iyz="-0.0" ixz="0.0"/>
-  </inertial>
-  <visual>
-    <origin xyz="0.006126 0.313823 -0.091838" rpy="0 0 0"/>
-    <geometry>
-      <mesh filename="file://$(find assem1_description)/meshes/lidar_1.STL" scale="0.001 0.001 0.001"/>
-    </geometry>
-    <material name="silver"/>
-  </visual>
-  <collision>
-    <origin xyz="0.006126 0.313823 -0.091838" rpy="0 0 0"/>
-    <geometry>
-      <mesh filename="file://$(find assem1_description)/meshes/lidar_1.STL" scale="0.001 0.001 0.001"/>
     </geometry>
   </collision>
@@ -410,8 +391,3 @@
   <child link="camera_1"/>
 </joint>
-<joint name="Rigid 17" type="fixed">
-  <origin xyz="-0.006126 -0.313823 0.091838" rpy="0 0 0"/>
-  <parent link="base_link"/>
-  <child link="lidar_1"/>
-</joint>
 </robot>

File: assem1_description/urdf/materials.xacro (robot description, xacro)
@@ -4,3 +4,6 @@
   <color rgba="0.700 0.700 0.700 1.000"/>
 </material>
+<material name="red">
+  <color rgba="1.0 0.0 0.0 1.0"/>
+</material>
 </robot>

Commit message: added camera

File: assem1_description/urdf/assem1.urdf.xacro (robot description, xacro)
@@ -4,4 +4,5 @@
 <xacro:include filename="$(find assem1_description)/urdf/assem1.gazebo" />
 <xacro:include filename="$(find assem1_description)/urdf/lidar.xacro"/>
+<xacro:include filename="$(find assem1_description)/urdf/camera.xacro"/>
 <link name="base_link">
   <inertial>
@@ -281,24 +282,4 @@
     <geometry>
       <mesh filename="file://$(find assem1_description)/meshes/wheel_v1__3__1.STL" scale="0.001 0.001 0.001"/>
-    </geometry>
-  </collision>
-</link>
-<link name="camera_1">
-  <inertial>
-    <origin xyz="-2.3577520093243098e-07 -0.005000272268811223 -4.671202445682976e-08" rpy="0 0 0"/>
-    <mass value="0.18839999999999998"/>
-    <inertia ixx="2.7e-05" iyy="8.2e-05" izz="5.8e-05" ixy="-0.0" iyz="-0.0" ixz="0.0"/>
-  </inertial>
-  <visual>
-    <origin xyz="0.003063 0.316911 -0.045919" rpy="0 0 0"/>
-    <geometry>
-      <mesh filename="file://$(find assem1_description)/meshes/camera_1.STL" scale="0.001 0.001 0.001"/>
-    </geometry>
-    <material name="silver"/>
-  </visual>
-  <collision>
-    <origin xyz="0.003063 0.316911 -0.045919" rpy="0 0 0"/>
-    <geometry>
-      <mesh filename="file://$(find assem1_description)/meshes/camera_1.STL" scale="0.001 0.001 0.001"/>
     </geometry>
   </collision>
@@ -386,8 +367,3 @@
   <axis xyz="1.0 0.0 0.0"/>
 </joint>
-<joint name="Rigid 16" type="fixed">
-  <origin xyz="-0.003063 -0.316911 0.045919" rpy="0 0 0"/>
-  <parent link="base_link"/>
-  <child link="camera_1"/>
-</joint>
 </robot>

Commit message: localized_map and slam implemented

File: assem1_description/urdf/assem1.urdf.xacro (robot description, xacro)
@@ -25,4 +25,11 @@
   </collision>
 </link>
+<joint name="base_footprint_joint" type="fixed">
+  <parent link="base_link"/>
+  <child link="base_footprint"/>
+  <origin xyz="0 0 0" rpy="0.0 0.0 0.0"/>
+</joint>
+<link name="base_footprint">
+</link>
 <link name="Part2_1">
   <inertial>

File: assem1_description/urdf/lidar.xacro (robot description, xacro)
@@ -2,5 +2,5 @@
 <robot xmlns:xacro="http://www.ros.org/wiki/xacro" >
     <joint name="Rigid 17" type="fixed">
-        <origin xyz="-0.006126 -0.313823 0.091838" rpy="0 0 0"/>
+        <origin xyz="-0.006126 -0.313823 0.091838" rpy="0 0 -0.75"/>
         <parent link="base_link"/>
         <child link="lidar_1"/>
@@ -38,5 +38,5 @@
                         <resolution>1</resolution>
                         <min_angle>-3.14</min_angle>
-                        <max_angle>3.14</max_angle>
+                        <max_angle>1.57</max_angle>
                     </horizontal>
                 </scan>
